File: pcb/logic-gate-calculator.kicad_pcb (KiCad board)
At the start: 2 copper layers, 67.9 x 71.8 mm, 77 parts, among them J1 Power_Dupont_Socket_Connector, SW21 SW_0_in_A, SW22 SW_1_in_A, SW23 SW_2_in_A, SW24 SW_3_in_A, SW25 SW_4_in_A, SW26 SW_5_in_A, SW27 SW_6_in_A, SW28 SW_7_in_A, SW29 SW_8_in_A, SW30 SW_9_in_A, SW31 SW_0_in_B, SW32 SW_1_in_B, SW33 SW_2_in_B, SW34 SW_3_in_B, SW35 SW_4_in_B, SW36 SW_5_in_B, SW37 SW_6_in_B, SW38 SW_7_in_B, SW39 SW_8_in_B, SW40 SW_9_in_B, U34 SN74HC04N, U35 SN74HC42N, U36 CD74HC147E, U37 CD74HC283E, U38 CD74HC147E, U39 SN74HC04N, U40 L7805

Commit message: finish pcb and upload gerbers and step
Parts:
- U34, U39: value SN74HC04N -> N14
- U35: value SN74HC42N -> N16
- U36, U38: value CD74HC147E -> N16
- U37: value CD74HC283E -> N16
- moved U35 148.0 mm to (182.3, 148.1)
- moved R35 144.5 mm to (167.6, 50.7)
- moved R50 137.2 mm to (167.5, 54.7)
- moved R48 132.1 mm to (167.6, 58.8)
- moved R49 132.1 mm to (167.6, 62.8)
- moved R32 128.5 mm to (154.8, 50.7)
- moved C8 126.9 mm to (184.8, 132.8), turned to 90 degrees
- moved R38 126.4 mm to (141.9, 50.7)
- moved R39 126.4 mm to (141.9, 54.7)
- moved R31 126.3 mm to (154.8, 54.7)
- moved SW33 126.0 mm to (175.1, 89.6)
- moved U34 124.3 mm to (144.5, 146.9)
- moved C7 120.2 mm to (172.2, 132.9), turned to 90 degrees
- moved SW36 119.4 mm to (175.1, 99.8)
- moved U37 118.9 mm to (169.8, 148.2)
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Connections:
- C8 pad 2: Net-(U35-VCC) -> +5V
- C9 pad 2: Net-(U35-VCC) -> 0_out
- R51 pad 1: Net-(U35-VCC) -> +5V
- R52 pad 1: Net-(U35-VCC) -> +5V
- R53 pad 1: Net-(U35-VCC) -> +5V
- R54 pad 1: Net-(U35-VCC) -> +5V
- R55 pad 1: Net-(U35-VCC) -> +5V
- R56 pad 1: Net-(U35-VCC) -> +5V
- R57 pad 1: Net-(U35-VCC) -> +5V
- R58 pad 1: Net-(U35-VCC) -> +5V
- R59 pad 1: Net-(U35-VCC) -> +5V
- R60 pad 1: Net-(U35-VCC) -> +5V
- U35 pad 16: Net-(U35-VCC) -> +5V
Routing:
- net +5V: track 0.00 -> 412.5 mm
- net 2_in_B: track 0.00 -> 170.7 mm, vias 0 -> 2
- net 1_in_A: track 0.00 -> 163.1 mm, vias 0 -> 4
- net 0_out: track 0.00 -> 157.3 mm, vias 0 -> 31
- net 9_in_B: track 0.00 -> 152.3 mm, vias 0 -> 2
- net 1_in_B: track 0.00 -> 142.6 mm, vias 0 -> 8
- net 5_in_B: track 0.00 -> 129.2 mm, vias 0 -> 4
- net 8_in_B: track 0.00 -> 127.8 mm, vias 0 -> 5
- net 2_in_A: track 0.00 -> 124.6 mm, vias 0 -> 2
- net 7_in_B: track 0.00 -> 122.1 mm, vias 0 -> 5
- net 4_in_A: track 0.00 -> 120.9 mm, vias 0 -> 6
- net LED_0: track 0.00 -> 120.7 mm, vias 0 -> 19
- net 8_in_A: track 0.00 -> 114.8 mm, vias 0 -> 1
- net 6_in_A: track 0.00 -> 113.3 mm, vias 0 -> 1
- net 7_in_A: track 0.00 -> 112.5 mm, vias 0 -> 5
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- added copper zone on B.Cu, net 0_out
Other:
- board size 67.9 x 71.8 mm -> 86 x 115 mm
- board text added: "+"
- board text added: "0"
- board text added: "1"
- board text added: "10kΩ"
- board text added: "2"
- board text added: "220Ω"
- board text added: "3"
- board text added: "4"
- board text added: "4-Bit Adder"
- board text added: "5"
- board text added: "6"
- board text added: "7"
- board text added: "8"
- board text added: "9"
- board text added: "A calculator that sums two 0-9 numbers into a 0-9 sum."
- board text added: "By Jayden Leung, 16 Boston"
- board text added: "Decoding"
- board text added: "Encoding A"
- board text added: "Encoding B"
- board text added: "Inverting A"
- board text added: "Inverting B"
- board text added: "Logic Gate Calculator"
- board text added: "Num 1"
- board text added: "Num 2"
- board text added: "Only sums ranging from 0-9 will be displayed."
- board text added: "Output Sum"
- board text added: "Power Input"
