File: pcb/logic-gate-calculator.kicad_pcb (KiCad board)
At the start: 2 copper layers, 86 x 115 mm, 77 parts, among them J1 Power_Dupont_Socket_Connector, SW21 SW_0_in_A, SW22 SW_1_in_A, SW23 SW_2_in_A, SW24 SW_3_in_A, SW25 SW_4_in_A, SW26 SW_5_in_A, SW27 SW_6_in_A, SW28 SW_7_in_A, SW29 SW_8_in_A, SW30 SW_9_in_A, SW31 SW_0_in_B, SW32 SW_1_in_B, SW33 SW_2_in_B, SW34 SW_3_in_B, SW35 SW_4_in_B, SW36 SW_5_in_B, SW37 SW_6_in_B, SW38 SW_7_in_B, SW39 SW_8_in_B, SW40 SW_9_in_B, U34 N14, U35 N16, U36 N16, U37 N16, U38 N16, U39 N14, U40 L7805

Commit message: fix numbering
Other:
- board text added: "*ESD Warning - board may malfunction if ungrounded."
