File: pcb/logic-gate-calculator.kicad_sch (KiCad schematic)
At the start: 234 parts, among them J1 Power_Dupont_Socket_Connector, Q1 BS170, Q12 BS170, Q13 BS170, Q14 BS170, Q15 BS170, Q18 BS170, Q19 BS170, Q2 BS170, Q20 BS170, Q21 BS170, Q3 BS170, Q4 BS170, Q5 BS170, Q6 BS170, Q7 BS170, Q8 BS170, Q9 BS170, SW1 SW_0_in_A, SW10 SW_9_in_A, SW11 SW_0_in_B, SW12 SW_1_in_B, SW13 SW_2_in_B, SW14 SW_3_in_B, SW15 SW_4_in, SW16 SW_5_in, SW17 SW_6_in_B, SW18 SW_7_in_B, SW19 SW_8_in_B, SW2 SW_1_in_A, SW20 SW_9_in_B, SW21 SW_0_in_A, SW22 SW_1_in_A, SW23 SW_2_in_A, SW24 SW_3_in_A, SW25 SW_4_in_A, SW26 SW_5_in_A, SW27 SW_6_in_A, SW28 SW_7_in_A, SW29 SW_8_in_A, SW3 SW_2_in_A, SW30 SW_9_in_A, SW31 SW_0_in_B, SW32 SW_1_in_B, SW33 SW_2_in_B, SW34 SW_3_in_B, SW35 SW_4_in_B, SW36 SW_5_in_B, SW37 SW_6_in_B, SW38 SW_7_in_B, SW39 SW_8_in_B, SW4 SW_3_in_A, SW40 SW_9_in_B, SW5 SW_4_in, SW6 SW_5_in, SW7 SW_6_in_A, SW8 SW_7_in_A, SW9 SW_8_in_A, U1 74LS86, U2 74LS08, U20 74LS21, U21 74LS21, U22 74LS21, U23 74LS21, U24 74LS21, U25 74LS21, U26 74LS21, U27 74LS21, U28 74LS21, U29 74LS21, U3 74LS86, U30 74AUC2G04, U31 74AUC2G04, U32 74AUC2G04, U33 74AUC2G04, U34 SN74HC04N, U35 SN74HC42N, U36 CD74HC147E, U37 CD74HC283E, U38 CD74HC147E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

Commit message: finish pcb and upload gerbers and step
Connections:
- net +5V: now also C8.2, R51.1, R52.1, R53.1, R54.1, R55.1, R56.1, R57.1, R58.1, R59.1, R60.1, U35.16 (VCC)
- net 0_out: now also C9.2
Other:
- moved on the sheet: C9
Changed lines of the file:
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@@
 	)
 	(junction
+		(at 215.9 378.46)
+		(diameter 0)
+		(color 0 0 0 0)
+	)
+	(junction
 		(at 167.64 111.76)
 		(diameter 0)
@@
 	)
 	(junction
-		(at 215.9 378.46)
+		(at 120.65 195.58)
 		(diameter 0)
 		(color 0 0 0 0)
 	)
 	(junction
-		(at 120.65 195.58)
+		(at 365.76 40.64)
 		(diameter 0)
 		(color 0 0 0 0)
 	)
 	(junction
-		(at 365.76 40.64)
+		(at 215.9 382.27)
 		(diameter 0)
 		(color 0 0 0 0)
@@
 	(wire
 		(pts
+			(xy 215.9 378.46) (xy 215.9 382.27)
+		)
+		(stroke
+			(width 0)
+			(type default)
+		)
+	)
+	(wire
+		(pts
 			(xy 414.02 119.38) (xy 421.64 119.38)
 		)
@@
 	(wire
 		(pts
+			(xy 215.9 382.27) (xy 215.9 386.08)
+		)
+		(stroke
+			(width 0)
+			(type default)
+		)
+	)
+	(wire
+		(pts
 			(xy 516.89 72.39) (xy 529.59 72.39)
 		)
@@
 	(wire
 		(pts
+			(xy 215.9 378.46) (xy 231.14 378.46)
+		)
+		(stroke
+			(width 0)
+			(type default)
+		)
+	)
+	(wire
+		(pts
 			(xy 511.81 62.23) (xy 511.81 67.31)
 		)
@@
 	(wire
 		(pts
-			(xy 215.9 378.46) (xy 231.14 378.46)
-		)
-		(stroke
-			(width 0)
-			(type default)
-		)
-	)
-	(wire
-		(pts
 			(xy 256.54 368.3) (xy 259.08 368.3)
 		)
@@
 	(symbol
 		(lib_id "Device:C")
-		(at 215.9 382.27 180)
+		(at 212.09 382.27 270)
 		(unit 1)
 		(exclude_from_sim no)
@@
 		(dnp no)
 		(property "Reference" "C9"
-			(at 207.01 381.254 0)
+			(at 211.582 389.128 90)
 			(effects
 				(font
@@
 		)
 		(property "Value" "2.2µF"
-			(at 207.01 383.794 0)
+			(at 211.582 386.588 90)
 			(effects
 				(font
@@
 		)
 		(property "Footprint" "Capacitor_THT:C_Disc_D6.0mm_W2.5mm_P5.00mm"
-			(at 214.9348 378.46 0)
+			(at 208.28 383.2352 0)
 			(effects
 				(font
@@
 		)
 		(property "Datasheet" "~"
-			(at 215.9 382.27 0)
+			(at 212.09 382.27 0)
 			(effects
 				(font
@@
 		)
 		(property "Description" "Unpolarized capacitor"
-			(at 215.9 382.27 0)
+			(at 212.09 382.27 0)
 			(effects
 				(font
@@
 					(unit 1)
 				)
+			)
+		)
+	)
+	(symbol
+		(lib_id "power:GND")
+		(at 208.28 382.27 270)
+		(unit 1)
+		(exclude_from_sim no)
+		(in_bom yes)
+		(on_board yes)
+		(dnp no)
+		(fields_autoplaced yes)
+		(property "Reference" "#PWR0278"
+			(at 201.93 382.27 0)
+			(effects
+				(font
+					(size 1.27 1.27)
+				)
+				(hide yes)
+			)
+		)
+		(property "Value" "GND"
+			(at 204.47 382.2699 90)
+			(effects
+				(font
+					(size 1.27 1.27)
+				)
+				(justify right)
+			)
+		)
+		(property "Footprint" ""
+			(at 208.28 382.27 0)
+			(effects
+				(font
+					(size 1.27 1.27)
+				)
+				(hide yes)
+			)
+		)
+		(property "Datasheet" ""
+			(at 208.28 382.27 0)
+			(effects
+				(font
+					(size 1.27 1.27)
+				)
+				(hide yes)
+			)
+		)
+		(property "Description" "Power symbol creates a global label with name \"GND\" , ground"
+			(at 208.28 382.27 0)
+			(effects
+				(font
+					(size 1.27 1.27)
+				)
+				(hide yes)
+			)
+		)
+		(pin "1"
+		)
+		(instances
+			(project "logic-gate-calculator"
+				(path "/9b79f451-5707-4d18-970a-918096944587"
+					(reference "#PWR0278")
+					(unit 1)
+				)
